Commit message: [canopies] Add data

File: examples/canopies/data/canopies_without_gripper.urdf (robot description, URDF)
Before this commit: robot canopies, 98 links, 97 joints
Links:
- removed link camera_support_left_link
- removed link camera_support_right_link
- removed link left_blade_arm_left
- removed link left_blade_arm_right
- removed link linear_actuator_1_left_input
- removed link linear_actuator_1_left_output
- removed link linear_actuator_1_right_input
- removed link linear_actuator_1_right_output
- removed link linear_actuator_2_left_input
- removed link linear_actuator_2_left_output
- removed link linear_actuator_2_right_input
- removed link linear_actuator_2_right_output
- removed link right_blade_arm_left
- removed link right_blade_arm_right
- added link bracelet_left_link, mass 0.00498877703130037; collision mesh filename=package://canopies_description/meshes/end-effector/camera_r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; visual mesh filename=package://canopies_description/meshes/end-effector/camera_r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
- added link bracelet_right_link, mass 0.00498877703130037; collision mesh filename=package://canopies_description/meshes/end-effector/camera_r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; visual mesh filename=package://canopies_description/meshes/end-effector/camera_r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
- added link sliding_camera_left_link, mass 0.045942703958924; collision mesh filename=package://canopies_description/meshes/end-effector/sliding_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; visual mesh filename=package://canopies_description/meshes/end-effector/sliding_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
- added link sliding_camera_right_link, mass 0.045942703958924; collision mesh filename=package://canopies_description/meshes/end-effector/sliding_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; visual mesh filename=package://canopies_description/meshes/end-effector/sliding_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
Joints:
- removed joint camera_support_left_joint
- removed joint camera_support_right_joint
- removed joint left_blade_arm_left_joint
- removed joint left_blade_arm_right_joint
- removed joint linear_actuator_1_left_input_joint
- removed joint linear_actuator_1_left_output_joint
- removed joint linear_actuator_1_right_input_joint
- removed joint linear_actuator_1_right_output_joint
- removed joint linear_actuator_2_left_input_joint
- removed joint linear_actuator_2_left_output_joint
- removed joint linear_actuator_2_right_input_joint
- removed joint linear_actuator_2_right_output_joint
- removed joint right_blade_arm_left_joint
- removed joint right_blade_arm_right_joint
- added joint bracelet_left_joint: type fixed, parent base_gripper_left_link, child bracelet_left_link, origin xyz=0 0 0 rpy=0 0 0
- added joint bracelet_right_joint: type fixed, parent base_gripper_right_link, child bracelet_right_link, origin xyz=0 0 0 rpy=0 0 0
- added joint sliding_camera_left_joint: type fixed, parent bracelet_left_link, child sliding_camera_left_link, origin xyz=0 0.05352 -0.032425 rpy=-1.5708 -1.5708 0
- added joint sliding_camera_right_joint: type fixed, parent bracelet_right_link, child sliding_camera_right_link, origin xyz=0 0.05352 -0.032425 rpy=-1.5708 -1.5708 0
- joint arm_left_7_joint: limit lower=-3.6 upper=1.3701 effort=50 velocity=1.95 -> lower=-2.5044 upper=2.5044 effort=50 velocity=1.95
- joint arm_right_7_joint: limit lower=-3.6 upper=1.3701 effort=50 velocity=1.95 -> lower=-2.5044 upper=2.5044 effort=50 velocity=1.95
- joint base_gripper_left_joint: origin xyz=0 0 -0.0005 rpy=0 0 0 -> xyz=0 0 -0.001 rpy=0 0 -1.117359787
- joint base_gripper_right_joint: origin xyz=0 0 0.0005 rpy=0 3.1415 0. -> xyz=0 0 0.001 rpy=0 3.1415 0.
- joint camera_left_d435_joint: parent camera_support_left_link -> sliding_camera_left_link
- joint camera_right_d435_joint: parent camera_support_right_link -> sliding_camera_right_link
- joint inner_finger_1_left_joint: origin xyz=0.013977 0.0125 0.13388 rpy=1.5708 -0.2618 -3.1416 -> xyz=0.014 0.011 0.07885 rpy=1.5708 -0.2618 -3.1416
- joint inner_finger_1_right_joint: origin xyz=0.013977 0.0125 0.13388 rpy=1.5708 -0.2618 -3.1416 -> xyz=0.014 0.011 0.07885 rpy=1.5708 -0.2618 -3.1416
- joint inner_finger_2_left_joint: origin xyz=-0.0139772762825847014 0.0124999999999999 0.133881761423197 rpy=1.5708 0.2618 -3.1416 -> xyz=-0.014 0.011 0.07885 rpy=1.5708 0.2618 -3.1416
- joint inner_finger_2_right_joint: origin xyz=-0.0139772762825847014 0.0124999999999999 0.133881761423197 rpy=1.5708 0.2618 -3.1416 -> xyz=-0.014 0.011 0.07885 rpy=1.5708 0.2618 -3.1416
- joint outer_finger_1_left_joint: origin xyz=0.0288 -0.00 0.12935 rpy=1.5708 -0.2618 3.1416 -> xyz=0.028823 -0.002 0.074318 rpy=1.5708 -0.2618 3.1416
- joint outer_finger_1_right_joint: origin xyz=0.0288 -0.00 0.12935 rpy=1.5708 -0.2618 3.1416 -> xyz=0.028823 -0.002 0.074318 rpy=1.5708 -0.2618 3.1416
- joint outer_finger_2_left_joint: origin xyz=-0.0288 -0.00 0.12935 rpy=1.5708 0.2618 -3.1416 -> xyz=-0.028823 -0.003 0.074318 rpy=1.5708 0.2618 -3.1416
- joint outer_finger_2_right_joint: origin xyz=-0.0288 -0.00 0.12935 rpy=1.5708 0.2618 -3.1416 -> xyz=-0.028823 -0.003 0.074318 rpy=1.5708 0.2618 -3.1416

File: examples/canopies/data/offset_test_sample.xacro (robot description, xacro)
@@ -1,16 +1,16 @@
-<xacro:property name="camera_position_x" value="0.090995804978574" / >
-<xacro:property name="camera_position_y" value="0.0809996288777572" / >
-<xacro:property name="camera_position_z" value="0.0022150984609048945" / >
-<xacro:property name="camera_orientation_r" value="-1.5699992598138324" / >
-<xacro:property name="camera_orientation_p" value="-3.133256816881189e-06" / >
-<xacro:property name="camera_orientation_y" value="1.7251181665387005e-07" / >
-<xacro:property name="head_2_joint_joint_offset" value="0.0046947909366622555" / >
-<xacro:property name="head_1_joint_joint_offset" value="0.004694137460690144" / >
-<xacro:property name="torso_lift_joint_joint_offset" value="-5.649668935744139e-06" / >
-<xacro:property name="arm_left_1_joint_joint_offset" value="-0.006573592400299189" / >
-<xacro:property name="arm_left_2_joint_joint_offset" value="0.04960260234675106" / >
-<xacro:property name="arm_left_3_joint_joint_offset" value="0.004379886888349329" / >
-<xacro:property name="arm_left_4_joint_joint_offset" value="-0.012860702297996894" / >
-<xacro:property name="arm_left_5_joint_joint_offset" value="0.02768534601594298" / >
-<xacro:property name="arm_left_6_joint_joint_offset" value="0.036215629330525544" / >
-<xacro:property name="arm_left_7_joint_joint_offset" value="-0.002258555594277815" / >
+<xacro:property name="camera_position_x" value="0.23352414041645495" / >
+<xacro:property name="camera_position_y" value="0.12494454999619337" / >
+<xacro:property name="camera_position_z" value="-0.028341878365666377" / >
+<xacro:property name="camera_orientation_r" value="-1.555457874388913" / >
+<xacro:property name="camera_orientation_p" value="-0.014199943575185994" / >
+<xacro:property name="camera_orientation_y" value="-0.12307665386463595" / >
+<xacro:property name="head_2_joint_joint_offset" value="-0.04384735011178917" / >
+<xacro:property name="head_1_joint_joint_offset" value="-0.04349985355802542" / >
+<xacro:property name="torso_lift_joint_joint_offset" value="0.00024608156936450014" / >
+<xacro:property name="arm_left_1_joint_joint_offset" value="-0.06703198834255336" / >
+<xacro:property name="arm_left_2_joint_joint_offset" value="0.0050212065091361" / >
+<xacro:property name="arm_left_3_joint_joint_offset" value="0.005911069400929951" / >
+<xacro:property name="arm_left_4_joint_joint_offset" value="0.021267132393414826" / >
+<xacro:property name="arm_left_5_joint_joint_offset" value="-0.04769672268820761" / >
+<xacro:property name="arm_left_6_joint_joint_offset" value="0.020596686911109892" / >
+<xacro:property name="arm_left_7_joint_joint_offset" value="-0.02523670109042842" / >
