Commit message: [tiago] change package path

File: examples/tiago/data/tiago.urdf (robot description, URDF)
Before this commit: robot tiago, 78 links, 77 joints
Links:
- link arm_1_link: geometry collision mesh filename=package://tiago_description/meshes/arm/arm_1_collision.dae scale=1 1 1; visual mesh filename=package://tiago_description/meshes/arm/arm_1.stl scale=1 1 1
- link arm_2_link: geometry collision mesh filename=package://tiago_description/meshes/arm/arm_2_collision.dae scale=1 1 1; visual mesh filename=package://tiago_description/meshes/arm/arm_2.stl scale=1 1 1
- link arm_3_link: geometry collision mesh filename=package://tiago_description/meshes/arm/arm_3_collision.dae scale=1 1 1; visual mesh filename=package://tiago_description/meshes/arm/arm_3.stl scale=1 1 1
- link arm_4_link: geometry collision mesh filename=package://tiago_description/meshes/arm/arm_4_collision.dae scale=1 1 1; visual mesh filename=package://tiago_description/meshes/arm/arm_4.stl scale=1 1 1
- link arm_5_link: geometry collision mesh filename=package://tiago_description/meshes/arm/arm_5_collision.dae scale=1 1 1; visual mesh filename=package://tiago_description/meshes/arm/arm_5.stl scale=1 1 1
- link arm_6_link: geometry collision mesh filename=package://tiago_description/meshes/arm/arm_6_collision.dae scale=1 1 1; visual mesh filename=package://tiago_description/meshes/arm/arm_6.stl scale=1 1 1
- link base_antenna_left_link: geometry collision cylinder length=0.17 radius=0.005; visual mesh filename=package://tiago_description/meshes/pmb2/objects/antenna.stl
- link base_antenna_right_link: geometry collision cylinder length=0.17 radius=0.005; visual mesh filename=package://tiago_description/meshes/pmb2/objects/antenna.stl
- link base_cover_link: geometry visual mesh filename=package://tiago_description/meshes/pmb2/base/base_ring.stl
- link base_link: geometry collision mesh filename=package://tiago_description/meshes/pmb2/base/base_collision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; visual mesh filename=package://tiago_description/meshes/pmb2/base/base.stl
- link caster_back_left_1_link: geometry visual mesh filename=package://tiago_description/meshes/pmb2/wheels/caster_1.stl
- link caster_back_left_2_link: geometry collision sphere radius=0.025; visual mesh filename=package://tiago_description/meshes/pmb2/wheels/caster_2.stl
- link caster_back_right_1_link: geometry visual mesh filename=package://tiago_description/meshes/pmb2/wheels/caster_1.stl
- link caster_back_right_2_link: geometry collision sphere radius=0.025; visual mesh filename=package://tiago_description/meshes/pmb2/wheels/caster_2.stl
- link caster_front_left_1_link: geometry visual mesh filename=package://tiago_description/meshes/pmb2/wheels/caster_1.stl
- link caster_front_left_2_link: geometry collision sphere radius=0.025; visual mesh filename=package://tiago_description/meshes/pmb2/wheels/caster_2.stl
- link caster_front_right_1_link: geometry visual mesh filename=package://tiago_description/meshes/pmb2/wheels/caster_1.stl
- link caster_front_right_2_link: geometry collision sphere radius=0.025; visual mesh filename=package://tiago_description/meshes/pmb2/wheels/caster_2.stl
- link hand_index_abd_link: geometry collision mesh filename=package://tiago_description/meshes/hey5/finger_abd_collisio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 scale=1 1 1; visual mesh filename=package://tiago_description/meshes/hey5/finger_abd_collisio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 scale=1 1 1
- link hand_index_flex_1_link: geometry collision mesh filename=package://tiago_description/meshes/hey5/finger_flex_collisi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; visual mesh filename=package://tiago_description/meshes/hey5/finger_flex_collisi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
- link hand_index_flex_2_link: geometry collision mesh filename=package://tiago_description/meshes/hey5/finger_flex_collisi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; visual mesh filename=package://tiago_description/meshes/hey5/finger_flex_collisi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
- link hand_index_flex_3_link: geometry collision mesh filename=package://tiago_description/meshes/hey5/finger_flex_tip_col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; visual mesh filename=package://tiago_description/meshes/hey5/finger_flex_tip_col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
- link hand_little_abd_link: geometry collision mesh filename=package://tiago_description/meshes/hey5/finger_abd_collisio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 scale=1 1 1; visual mesh filename=package://tiago_description/meshes/hey5/finger_abd_collisio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 scale=1 1 1
- link hand_little_flex_1_link: geometry collision mesh filename=package://tiago_description/meshes/hey5/finger_flex_collisi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; visual mesh filename=package://tiago_description/meshes/hey5/finger_flex_collisi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
- link hand_little_flex_2_link: geometry collision mesh filename=package://tiago_description/meshes/hey5/finger_flex_collisi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; visual mesh filename=package://tiago_description/meshes/hey5/finger_flex_collisi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
- link hand_little_flex_3_link: geometry collision mesh filename=package://tiago_description/meshes/hey5/finger_flex_tip_col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; visual mesh filename=package://tiago_description/meshes/hey5/finger_flex_tip_col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
- link hand_middle_abd_link: geometry collision mesh filename=package://tiago_description/meshes/hey5/finger_abd_collisio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 scale=1 1 1; visual mesh filename=package://tiago_description/meshes/hey5/finger_abd_collisio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 scale=1 1 1
- link hand_middle_flex_1_link: geometry collision mesh filename=package://tiago_description/meshes/hey5/finger_flex_collisi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; visual mesh filename=package://tiago_description/meshes/hey5/finger_flex_collisi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
- link hand_middle_flex_2_link: geometry collision mesh filename=package://tiago_description/meshes/hey5/finger_flex_collisi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; visual mesh filename=package://tiago_description/meshes/hey5/finger_flex_collisi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
- link hand_middle_flex_3_link: geometry collision mesh filename=package://tiago_description/meshes/hey5/finger_flex_tip_col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; visual mesh filename=package://tiago_description/meshes/hey5/finger_flex_tip_col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
- link hand_palm_link: geometry collision mesh filename=package://tiago_description/meshes/hey5/palm_collision.stl scale=1 1 1; visual mesh filename=package://tiago_description/meshes/hey5/palm.stl scale=1 1 1
- link hand_ring_abd_link: geometry collision mesh filename=package://tiago_description/meshes/hey5/finger_abd_collisio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 scale=1 1 1; visual mesh filename=package://tiago_description/meshes/hey5/finger_abd_collisio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 scale=1 1 1
- link hand_ring_flex_1_link: geometry collision mesh filename=package://tiago_description/meshes/hey5/finger_flex_collisi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; visual mesh filename=package://tiago_description/meshes/hey5/finger_flex_collisi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
- link hand_ring_flex_2_link: geometry collision mesh filename=package://tiago_description/meshes/hey5/finger_flex_collisi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; visual mesh filename=package://tiago_description/meshes/hey5/finger_flex_collisi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
- link hand_ring_flex_3_link: geometry collision mesh filename=package://tiago_description/meshes/hey5/finger_flex_tip_col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; visual mesh filename=package://tiago_description/meshes/hey5/finger_flex_tip_col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
- link hand_thumb_abd_link: geometry collision mesh filename=package://tiago_description/meshes/hey5/thumb_abd_collision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 scale=1 1 1; visual mesh filename=package://tiago_description/meshes/hey5/thumb_abd_collision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 scale=1 1 1
- link hand_thumb_flex_1_link: geometry collision mesh filename=package://tiago_description/meshes/hey5/finger_flex_collisi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; visual mesh filename=package://tiago_description/meshes/hey5/finger_flex_collisi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
- link hand_thumb_flex_2_link: geometry collision mesh filename=package://tiago_description/meshes/hey5/finger_flex_tip_col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; visual mesh filename=package://tiago_description/meshes/hey5/finger_flex_tip_col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
- link head_1_link: geometry collision mesh filename=package://tiago_description/meshes/head/head_1_collision.dae scale=1 1 1; visual mesh filename=package://tiago_description/meshes/head/head_1.stl scale=1 1 1
- link head_2_link: geometry collision mesh filename=package://tiago_description/meshes/head/head_2_collision.dae scale=1 1 1; visual mesh filename=package://tiago_description/meshes/head/head_2.stl scale=1 1 1
- link torso_fixed_link: geometry collision box size=0.25 0.25 0.1; collision box size=0.4 0.25 0.04
- link torso_lift_link: geometry collision mesh filename=package://tiago_description/meshes/torso/torso_lift_collisi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 scale=1 1 1; collision mesh filename=package://tiago_description/meshes/torso/torso_lift_collisi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 scale=1 1 1
- link wheel_left_link: geometry collision cylinder length=0.04 radius=0.0985; visual mesh filename=package://tiago_description/meshes/pmb2/wheels/wheel.stl
- link wheel_right_link: geometry collision cylinder length=0.04 radius=0.0985; visual mesh filename=package://tiago_description/meshes/pmb2/wheels/wheel.stl
