Commit message: [exemples][human]add human exemple until SIP (that must be revised at that stage)

File: models/others/robots/human_description/urdf/human.urdf (robot description, URDF)
Before this commit: robot human_36dof_ISB_model, 37 links, 36 joints
Links:
- link left_foot: geometry visual mesh filename=package://human_description/meshes/foot_mesh.STL scale=0.0060 0.0060 0.0060
- link left_hand: geometry visual mesh filename=package://human_description/meshes/hand_mesh.STL scale=0.0060 0.0060 0.0060
- link left_lowerarm: geometry visual mesh filename=package://human_description/meshes/lowerarm_mesh.STL scale=0.0060 0.0060 0.0060
- link left_lowerarm_virtual: geometry visual mesh filename=package://human_description/meshes/elbow_mesh.STL scale=0.0055 0.0055 0.0055
- link left_lowerleg: geometry visual mesh filename=package://human_description/meshes/lowerleg_mesh.STL scale=0.0063 0.0065 0.007
- link left_upperarm: geometry visual mesh filename=package://human_description/meshes/upperarm_mesh.STL scale=0.0063 0.0060 0.007
- link left_upperarm_virtual: geometry visual mesh filename=package://human_description/meshes/shoulder_mesh.STL scale=0.0055 0.0055 0.0055
- link left_upperleg: geometry visual mesh filename=package://human_description/meshes/upperleg_mesh.STL scale=0.0063 0.0065 0.007
- link left_upperleg_virtual_2: geometry visual mesh filename=package://human_description/meshes/knee_mesh.STL scale=0.006 0.006 0.006
- link middle_abdomen: geometry visual mesh filename=package://human_description/meshes/abdomen_mesh.STL scale=0.0055 0.0055 0.0055
- link middle_head: geometry visual mesh filename=package://human_description/meshes/head_mesh.STL scale=0.0055 0.0055 0.0055
- link middle_head_virtual: geometry visual mesh filename=package://human_description/meshes/neck_mesh.STL scale=0.005 0.005 0.005
- link middle_pelvis: geometry visual mesh filename=package://human_description/meshes/pelvis_mesh.STL scale=0.006 0.0055 0.0055
- link middle_thorax: geometry visual mesh filename=package://human_description/meshes/torso_mesh.STL scale=0.0065 0.0065 0.0065
- link right_foot: geometry visual mesh filename=package://human_description/meshes/foot_mesh.STL scale=0.0060 0.0060 0.0060
- link right_hand: geometry visual mesh filename=package://human_description/meshes/hand_mesh.STL scale=0.0060 0.0060 0.0060
- link right_lowerarm: geometry visual mesh filename=package://human_description/meshes/lowerarm_mesh.STL scale=0.0060 0.0060 0.0060
- link right_lowerarm_virtual: geometry visual mesh filename=package://human_description/meshes/elbow_mesh.STL scale=0.0055 0.0055 0.0055
- link right_lowerleg: geometry visual mesh filename=package://human_description/meshes/lowerleg_mesh.STL scale=0.0063 0.0065 0.007
- link right_upperarm: geometry visual mesh filename=package://human_description/meshes/upperarm_mesh.STL scale=0.0063 0.0060 0.007
- link right_upperarm_virtual: geometry visual mesh filename=package://human_description/meshes/shoulder_mesh.STL scale=0.0055 0.0055 0.0055
- link right_upperleg: geometry visual mesh filename=package://human_description/meshes/upperleg_mesh.STL scale=0.0063 0.0065 0.007
- link right_upperleg_virtual_2: geometry visual mesh filename=package://human_description/meshes/knee_mesh.STL scale=0.006 0.006 0.006

Commit message: [model] update the human model

File: models/others/robots/human_description/urdf/human.urdf (robot description, URDF)
Before this commit: robot human_36dof_ISB_model, 37 links, 36 joints
Links:
- added link base_link, mass 1e-6
- added link middle_abdomen_virtual_2
- added link middle_pelvis_virtual
- link left_clavicle: mass None -> 0.15600
- link left_foot: mass 1.13208 -> 0.86; geometry visual mesh filename=package://human_urdf/meshes/foot_mesh.STL scale=0.0060 0.0060 0.0060
- link left_hand: mass 0.56604 -> 0.43; geometry visual mesh filename=package://human_urdf/meshes/hand_mesh.STL scale=0.0060 0.0060 0.0060
- link left_lowerarm: mass 1.60378 -> 1.22; geometry visual mesh filename=package://human_urdf/meshes/lowerarm_mesh.STL scale=0.0060 0.0060 0.0060
- link left_lowerarm_virtual: geometry visual mesh filename=package://human_urdf/meshes/elbow_mesh.STL scale=0.0055 0.0055 0.0055
- link left_lowerleg: mass 4.52832 -> 3.45; geometry visual mesh filename=package://human_urdf/meshes/lowerleg_mesh.STL scale=0.0063 0.0065 0.007
- link left_upperarm: mass 2.26416 -> 1.73; geometry visual mesh filename=package://human_urdf/meshes/upperarm_mesh.STL scale=0.0063 0.0060 0.007
- link left_upperarm_virtual: geometry visual mesh filename=package://human_urdf/meshes/shoulder_mesh.STL scale=0.0055 0.0055 0.0055
- link left_upperleg: mass 11.6038 -> 8.84; geometry visual mesh filename=package://human_urdf/meshes/upperleg_mesh.STL scale=0.0063 0.0065 0.007
- link left_upperleg_virtual_2: geometry visual mesh filename=package://human_urdf/meshes/knee_mesh.STL scale=0.006 0.006 0.006
- link middle_abdomen: mass 2.73586 -> 1.94; geometry visual mesh filename=package://human_urdf/meshes/abdomen_mesh.STL scale=0.0055 0.0055 0.0055
- link middle_head: mass 6.32078 -> 4.82; geometry visual mesh filename=package://human_urdf/meshes/head_mesh.STL scale=0.0055 0.0055 0.0055
- link middle_head_virtual: geometry visual mesh filename=package://human_urdf/meshes/neck_mesh.STL scale=0.005 0.005 0.005
- link middle_pelvis: mass 13.3963 -> 10.21; geometry visual mesh filename=package://human_urdf/meshes/pelvis_mesh.STL scale=0.006 0.0055 0.0055
- link middle_thorax: mass 28.6794 -> 21.86; geometry visual mesh filename=package://human_urdf/meshes/torso_mesh.STL scale=0.0065 0.0065 0.0065
- link right_clavicle: mass None -> 0.15600
- link right_foot: mass 1.13208 -> 0.86; geometry visual mesh filename=package://human_urdf/meshes/foot_mesh.STL scale=0.0060 0.0060 0.0060
- link right_hand: mass 0.56604 -> 0.43; geometry visual mesh filename=package://human_urdf/meshes/hand_mesh.STL scale=0.0060 0.0060 0.0060
- link right_lowerarm: mass 1.60378 -> 1.22; geometry visual mesh filename=package://human_urdf/meshes/lowerarm_mesh.STL scale=0.0060 0.0060 0.0060
- link right_lowerarm_virtual: geometry visual mesh filename=package://human_urdf/meshes/elbow_mesh.STL scale=0.0055 0.0055 0.0055
- link right_lowerleg: mass 4.52832 -> 3.45; geometry visual mesh filename=package://human_urdf/meshes/lowerleg_mesh.STL scale=0.0063 0.0065 0.007
- link right_upperarm: mass 2.26416 -> 1.73; geometry visual mesh filename=package://human_urdf/meshes/upperarm_mesh.STL scale=0.0063 0.0060 0.007
- link right_upperarm_virtual: geometry visual mesh filename=package://human_urdf/meshes/shoulder_mesh.STL scale=0.0055 0.0055 0.0055
- link right_upperleg: mass 11.6038 -> 8.84; geometry visual mesh filename=package://human_urdf/meshes/upperleg_mesh.STL scale=0.0063 0.0065 0.007
- link right_upperleg_virtual_2: geometry visual mesh filename=package://human_urdf/meshes/knee_mesh.STL scale=0.006 0.006 0.006
Joints:
- added joint middle_abdomen_X: type revolute, parent middle_abdomen_virtual, child middle_abdomen_virtual_2, origin xyz=0 0 0 rpy=0 -0 0, axis 1 0 0, limit lower=-1.0472 upper=1.0472 effort=0 velocity=0
- added joint middle_abdomen_Y: type revolute, parent middle_abdomen_virtual_2, child middle_abdomen, origin xyz=0 0 0 rpy=0 -0 0, axis 0 1 0, limit lower=-1.0472 upper=1.0472 effort=0 velocity=0
- added joint middle_abdomen_Z: type revolute, parent middle_pelvis, child middle_abdomen_virtual, origin xyz=0.0 0.092 0.0 rpy=0 -0 0, axis 0 0 -1, limit lower=-1.0472 upper=0.392699 effort=0 velocity=0
- joint left_ankle_Z: origin xyz=0 -0.42805 0 rpy=0 -0 0 -> xyz=0.0 -0.421 0.0 rpy=0 -0 0
- joint left_clavicle_joint_X: origin xyz=0 0.330225 0 rpy=0 -0 0 -> xyz=0.0 0.319 0.0 rpy=0 -0 0
- joint left_elbow_Z: origin xyz=0 -0.2737 0 rpy=0 -0 0 -> xyz=0.0 -0.263 0.0 rpy=0 -0 0
- joint left_hip_X: axis -1 0 0 -> 1 0 0
- joint left_hip_Y: axis 0 -1 0 -> 0 1 0
- joint left_hip_Z: origin xyz=0.053375 -0.0749 -0.079975 rpy=0 -0 0 -> xyz=0.055 -0.077 -0.083 rpy=0 -0 0; parent middle_pelvis -> base_link
- joint left_knee: origin xyz=0 -0.427 0 rpy=0 -0 0 -> xyz=0.0 -0.42 0.0 rpy=0 -0 0
- joint left_shoulder_X: axis -1 0 0 -> 1 0 0
- joint left_shoulder_Y: axis 0 -1 0 -> 0 1 0; child left_upperarm_virtual -> left_upperarm; limit lower=-2.0944 upper=0.392699 effort=0 velocity=0 -> lower=-1.5708 upper=3.14159 effort=0 velocity=0; origin xyz=0.00805 -0.0728 -0.2037 rpy=0 -0 0 -> xyz=0 0 0 rpy=0 -0 0; parent left_clavicle -> left_upperarm_virtual_2
- joint left_shoulder_Z: child left_upperarm -> left_upperarm_virtual; limit lower=-1.5708 upper=3.14159 effort=0 velocity=0 -> lower=-2.0944 upper=0.392699 effort=0 velocity=0; origin xyz=0 0 0 rpy=0 -0 0 -> xyz=0.008 -0.075 -0.211 rpy=0 -0 0; parent left_upperarm_virtual_2 -> left_clavicle
- joint left_wrist_Z: origin xyz=0 -0.27965 0 rpy=0 -0 0 -> xyz=0.0 -0.275 0.0 rpy=0 -0 0
- joint middle_cervical_Z: axis 0 0 1 -> 0 0 -1; origin xyz=0 0.330225 0 rpy=0 -0 0 -> xyz=0.0 0.319 0.0 rpy=0 -0 0
- joint middle_lumbar_X: child middle_abdomen -> middle_pelvis; parent middle_abdomen_virtual -> middle_pelvis_virtual
- joint middle_lumbar_Z: axis 0 0 1 -> 0 0 -1; child middle_abdomen_virtual -> middle_pelvis_virtual; origin xyz=0 0 0 rpy=0 -0 0 -> xyz=0.0 0.0 0.0 rpy=0 -0 0; parent middle_pelvis -> base_link
- joint middle_thoracic_Z: axis 0 0 1 -> 0 0 -1; origin xyz=0 0.149275 0 rpy=0 -0 0 -> xyz=0.0 0.144 0.0 rpy=0 -0 0; parent middle_abdomen -> middle_pelvis
- joint right_ankle_Z: origin xyz=0 -0.42805 0 rpy=0 -0 0 -> xyz=0.0 -0.421 0.0 rpy=0 -0 0
- joint right_clavicle_joint_X: origin xyz=0 0.330225 0 rpy=0 -0 0 -> xyz=0.0 0.319 0.0 rpy=0 -0 0
- joint right_elbow_Z: origin xyz=0 -0.2737 0 rpy=0 -0 0 -> xyz=0.0 -0.263 0.0 rpy=0 -0 0
- joint right_hip_X: axis 1 0 0 -> -1 0 0
- joint right_hip_Y: axis 0 1 0 -> 0 -1 0
- joint right_hip_Z: origin xyz=0.053375 -0.0749 0.079975 rpy=0 -0 0 -> xyz=0.055 -0.077 0.083 rpy=0 -0 0; parent middle_pelvis -> base_link
- joint right_knee: origin xyz=0 -0.427 0 rpy=0 -0 0 -> xyz=0.0 -0.42 0.0 rpy=0 -0 0
- joint right_shoulder_X: axis 1 0 0 -> -1 0 0
- joint right_shoulder_Y: axis 0 1 0 -> 0 -1 0; child right_upperarm_virtual -> right_upperarm; limit lower=-2.0944 upper=0.392699 effort=0 velocity=0 -> lower=-1.5708 upper=3.14159 effort=0 velocity=0; origin xyz=0.00805 -0.0728 0.2037 rpy=0 -0 0 -> xyz=0 0 0 rpy=0 -0 0; parent right_clavicle -> right_upperarm_virtual_2
- joint right_shoulder_Z: child right_upperarm -> right_upperarm_virtual; limit lower=-1.5708 upper=3.14159 effort=0 velocity=0 -> lower=-2.0944 upper=0.392699 effort=0 velocity=0; origin xyz=0 0 0 rpy=0 -0 0 -> xyz=0.008 -0.075 0.211 rpy=0 -0 0; parent right_upperarm_virtual_2 -> right_clavicle
- joint right_wrist_Z: origin xyz=0 -0.27965 0 rpy=0 -0 0 -> xyz=0.0 -0.275 0.0 rpy=0 -0 0
